File: schematic/old_eagle/dust_sensor/dust_sensor.brd (EAGLE design)
At the start: 160 x 100 mm, 23 parts, among them IC1 LM1117T-5.0

Commit message: Mainboard
Parts:
- removed ANALOG1, ANALOG2, ANALOG3, ANALOG4, ANALOG5, ANALOG6, ANALOG7, DIGITAL1, DIGITAL2, DIGITAL3, DIGITAL4, DIGITAL5, DIGITAL6, DIGITAL7, DIGITAL8, UART1, UART2, UART3: (no value), SparkFun-Connectors:1X04
- removed C2: 100uF, resistor:C025-025X050
- removed IC1: LM1117T-5.0, lm1117:TO220
- removed STM32F411DISC: STM32F411_DISCOVERY, STM32F411_DISCOVERY:STM32F411_DISCOVERY
- added DUST_SENSOR: GP2Y1010AU0F, parts:GP2Y1010AU0F
- added R1: 150, SparkFun-Resistors:AXIAL-0.3
- added U$1: (no value), oshw:OSHW_8MM
- C1: value 10uF -> 220uF; device resistor:C025-025X050 -> resistor:E2,5-6
- J1: value (none) -> CONNECTOR; device con-jack:DCJ0303 -> SparkFun-Connectors:MOLEX-1X4
- moved J1 333.5 mm to (48.3, 66.0)
- moved C1 310.8 mm to (16.5, 66.0)
Connections:
- removed net ADC1: ANALOG1.3, STM32F411DISC.P$31
- removed net ADC10: ANALOG5.2, STM32F411DISC.P$4
- removed net ADC11: ANALOG6.3, STM32F411DISC.P$30
- removed net ADC12: ANALOG6.2, STM32F411DISC.P$5
- removed net ADC13: ANALOG7.3, STM32F411DISC.P$35
- removed net ADC14: ANALOG7.2, STM32F411DISC.P$10
- removed net ADC2: ANALOG1.2, STM32F411DISC.P$6
- removed net ADC3: ANALOG2.3, STM32F411DISC.P$33
- removed net ADC4: ANALOG2.2, STM32F411DISC.P$8
- removed net ADC5: ANALOG3.3, STM32F411DISC.P$34
- removed net ADC6: ANALOG3.2, STM32F411DISC.P$9
- removed net ADC7: ANALOG4.3, STM32F411DISC.P$36
- removed net ADC8: ANALOG4.2, STM32F411DISC.P$11
- removed net ADC9: ANALOG5.3, STM32F411DISC.P$29
- removed net CLK_1: DIGITAL1.2, STM32F411DISC.P$59
- removed net CLK_2: DIGITAL2.2, STM32F411DISC.P$84
- removed net CLK_3: DIGITAL3.2, STM32F411DISC.P$58
- removed net CLK_4: DIGITAL4.2, STM32F411DISC.P$83
- removed net CLK_5: DIGITAL5.2, STM32F411DISC.P$56
- removed net CLK_6: DIGITAL6.2, STM32F411DISC.P$13
- removed net CLK_7: DIGITAL7.2, STM32F411DISC.P$38
- removed net CLK_8: DIGITAL8.2, STM32F411DISC.P$14
- removed net DATA_1: DIGITAL1.3, STM32F411DISC.P$93
- removed net DATA_2: DIGITAL2.3, STM32F411DISC.P$67
- removed net DATA_3: DIGITAL3.3, STM32F411DISC.P$92
- removed net DATA_4: DIGITAL4.3, STM32F411DISC.P$66
- removed net DATA_5: DIGITAL5.3, STM32F411DISC.P$90
- removed net DATA_6: DIGITAL6.3, STM32F411DISC.P$64
- removed net DATA_7: DIGITAL7.3, STM32F411DISC.P$45
- removed net DATA_8: DIGITAL8.3, STM32F411DISC.P$21
- removed net IN_VCC: C1.1, IC1.3, J1.1
- removed net N$14: STM32F411DISC.P$101, STM32F411DISC.P$102
- removed net RX1: STM32F411DISC.P$87, UART1.3
- removed net RX2: STM32F411DISC.P$7, UART2.3
- removed net RX3: STM32F411DISC.P$99, UART3.3
- removed net TX1: STM32F411DISC.P$62, UART1.2
- removed net TX2: STM32F411DISC.P$32, UART2.2
- removed net TX3: STM32F411DISC.P$74, UART3.2
- new net DUST_OUT: DUST_SENSOR.VO, J1.3
- new net LED_CTRL: DUST_SENSOR.LED, J1.2
- net GND: now also C1.-, DUST_SENSOR.LED-GND, DUST_SENSOR.S-GND, J1.1; no longer ANALOG1.1, ANALOG2.1, ANALOG3.1, ANALOG4.1, ANALOG5.1, ANALOG6.1, ANALOG7.1, C1.2, C2.2, DIGITAL1.1, DIGITAL2.1, DIGITAL3.1, DIGITAL4.1, DIGITAL5.1, DIGITAL6.1, DIGITAL7.1, DIGITAL8.1, IC1.1, J1.2, J1.3, STM32F411DISC.P$1, STM32F411DISC.P$100, STM32F411DISC.P$12, STM32F411DISC.P$25, STM32F411DISC.P$26, STM32F411DISC.P$3, STM32F411DISC.P$50, STM32F411DISC.P$51, STM32F411DISC.P$75, STM32F411DISC.P$76, UART1.1, UART2.1, UART3.1
- net N$1: now also C1.+, DUST_SENSOR.V-LED, R1.P$2; no longer STM32F411DISC.P$103, STM32F411DISC.P$104
- net VCC: now also DUST_SENSOR.VCC, J1.4, R1.P$1; no longer ANALOG1.4, ANALOG2.4, ANALOG3.4, ANALOG4.4, ANALOG5.4, ANALOG6.4, ANALOG7.4, C2.1, DIGITAL1.4, DIGITAL2.4, DIGITAL3.4, DIGITAL4.4, DIGITAL5.4, DIGITAL6.4, DIGITAL7.4, DIGITAL8.4, IC1.2, STM32F411DISC.P$52, STM32F411DISC.P$77, UART1.4, UART2.4, UART3.4
Routing:
- net DUST_OUT: track 0.00 -> 142.9 mm
- net LED_CTRL: track 0.00 -> 129.4 mm
- net GND: track 0.00 -> 119.3 mm
- net VCC: track 0.00 -> 102.4 mm
- net N$1: track 0.00 -> 62.0 mm
- added copper zone on layer 1, net GND
Other:
- board size 160 x 100 mm -> 53.3 x 72.4 mm
- board text added: "Plug & Create Dust sensor module v1 https://tuankiet65.moe"
