File: schematic/main_board/main_board.kicad_pcb (KiCad board)
At the start: 2 copper layers, 101 x 67.3 mm, 69 parts, among them J1 UART_1, J10 I2C_2, J11 I2C_3, J12 I2C_4, J13 USB_OTG, J14 ANALOG, J15 SWD, J17 Barrel_Jack, J2 UART_2, J3 UART_3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

Commit message: Committing everything
Because my hard drive will soon crash and burn.o
Parts:
- added C18: 100n, Capacitors_SMD:C_1206_HandSoldering, B.Cu at (125.7, 79.4)
- added C19: 100n, Capacitors_SMD:C_1206_HandSoldering, B.Cu at (193.7, 78.1)
- added C20: 100n, Capacitors_SMD:C_1206_HandSoldering, B.Cu at (193.7, 94.6)
- added C21: 100n, Capacitors_SMD:C_1206_HandSoldering, B.Cu at (193.7, 111.1)
- added C22: 100n, Capacitors_SMD:C_1206_HandSoldering, B.Cu at (193.7, 127.6)
- added C23: 100n, Capacitors_SMD:C_1206_HandSoldering, B.Cu at (175.3, 123.8)
- added C24: 100n, Capacitors_SMD:C_1206_HandSoldering, B.Cu at (158.8, 123.8)
- added C25: 100n, Capacitors_SMD:C_1206_HandSoldering, B.Cu at (142.2, 123.8)
- added C26: 100n, Capacitors_SMD:C_1206_HandSoldering, B.Cu at (125.7, 123.8)
- added C27: 100n, Capacitors_SMD:C_1206_HandSoldering, B.Cu at (108.0, 127.6)
- added C28: 100n, Capacitors_SMD:C_1206_HandSoldering, B.Cu at (107.3, 111.1)
- added C29: 100n, Capacitors_SMD:C_1206_HandSoldering, B.Cu at (107.3, 94.6)
- added C30: 100n, Capacitors_SMD:C_1206_HandSoldering, B.Cu at (107.3, 78.1)
- added D7: SS34, Diodes_SMD:D_SMB, F.Cu at (167.0, 81.3)
- D5: value 3V3_LED_GREEN -> GREEN
- moved R6 8.60 mm to (165.7, 71.6)
- moved D6 8.55 mm to (168.8, 71.6)
- moved R13 4.19 mm to (148.5, 89.2)
- moved J13 3.05 mm to (158.6, 72.5)
- moved R19 2.16 mm to (148.5, 92.3)
- moved J12 1.31 mm to (111.1, 123.8)
- moved G*** 1.27 mm to (154.9, 95.9)
- moved C10 1.27 mm to (128.3, 99.9)
- moved C3 1.27 mm to (137.8, 99.9)
- moved C7 1.27 mm to (141.0, 99.9)
- moved C8 1.27 mm to (134.6, 99.9)
- moved C9 1.27 mm to (144.1, 99.9)
- moved L1 1.27 mm to (131.4, 99.9)
- moved J8 1.27 mm to (171.4, 120.7)
- moved R10 1.14 mm to (156.9, 89.0)
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Connections:
- C10 pad 1: Net-(C10-Pad1) -> VDDA
- C11 pad 1: Net-(C10-Pad1) -> VDDA
- J17 pad 1: Net-(C1-Pad1) -> Net-(D7-Pad2)
- L1 pad 2: Net-(C10-Pad1) -> VDDA
- R1 pad 1: +3V3 -> Net-(D5-Pad2)
- R1 pad 2: Net-(D5-Pad2) -> +3V3
- R13 pad 1: +5V -> +3V3
- R19 pad 1: +5V -> +3V3
- U1 pad 10: (no net) -> Net-(U1-Pad10)
- U1 pad 13: +3V3 -> VDDA
- U1 pad 2: (no net) -> Net-(U1-Pad2)
- U1 pad 3: (no net) -> /LSE_IN
- U1 pad 38: (no net) -> Net-(U1-Pad38)
- U1 pad 39: (no net) -> /MICROSD_D0
- U1 pad 4: (no net) -> /LSE_OUT
- U1 pad 40: (no net) -> /MICROSD_D1
- U1 pad 50: (no net) -> Net-(U1-Pad50)
- U1 pad 51: (no net) -> /MICROSD_D2
- U1 pad 53: (no net) -> /MICROSD_CLK
- U1 pad 54: (no net) -> /MICROSD_CMD
- U1 pad 56: (no net) -> Net-(U1-Pad56)
- U1 pad 8: (no net) -> Net-(U1-Pad8)
- U1 pad 9: (no net) -> Net-(U1-Pad9)
Routing:
- net GND: track 588.3 -> 711.1 mm, vias 4 -> 36
- net /BOOT0: track 67.5 -> 116.7 mm, vias 3 -> 2
- net /USB_ID: track 31.8 -> 79.7 mm, vias 3 -> 2
- net +5V: track 331.4 -> 368.9 mm, vias 2 -> 0
- net +3V3: track 157.8 -> 177.2 mm
- net /I2C1_SDA: track 107.5 -> 125.7 mm
- net /TX1: track 62.9 -> 79.5 mm
- net /RX1: track 64.9 -> 80.1 mm
- net /NRST: track 69.4 -> 83.2 mm, vias 2 -> 4
- net VDDA: track 0.00 -> 13.0 mm, vias 0 -> 1
- net /TX2: track 125.8 -> 138.2 mm
- net Net-(D7-Pad2): track 0.00 -> 12.1 mm
- net /RX2: track 132.3 -> 143.2 mm
- net /I2C1_SCL: track 111.0 -> 100.6 mm
- net Net-(C10-Pad1): track 7.62 -> 0.00 mm
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Other:
- board size 101 x 67.3 mm -> 100.3 x 67.3 mm
- board text added: "+"
- board text added: "-"
- board text added: "DC 9V-15V ONLY"
- board text added: "Plug & Create"
- board text added: "Plug & Create Mainboard v3 based on the PyBoard v1.1 running MicroPython Made by Ho Tuan Kiet https://tuankiet65.moe KiCad sources available on GitHub: tuankiet65/pnc-modules"
- board text added: "[USB signal tracks]"
- board text removed: "DC 9V-12V ONLY"
- board text removed: "Plug & Play"
- board text removed: "Plug & Play Mainboard v3 Made by Ho Tuan Kiet https://tuankiet65.moe Based on the PyBoard v1.1 by the MicroPython Project KiCad sources available on GitHub: tuankiet65/pnc-modules"
