File: schematic/old_eagle/main_board/main_board.sch (EAGLE design)
At the start: 16 parts, among them IC1 LM1117MPX-5.0, J1 POWER_JACK, U1 STM32L151C6T6

Commit message: Committing everything
Because my hard drive will soon crash and burn.o
Parts:
- removed JP1: (no value), pinhead:PINHD-1X12
- removed U1: STM32L151C6T6, ST Microelctronics_By_element14_Batch_1:STM32L151C6T6
Changed lines of the file:
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@@
 <?xml version="1.0" encoding="utf-8"?>
 <!DOCTYPE eagle SYSTEM "eagle.dtd">
-<eagle version="8.3.1">
+<eagle version="8.5.2">
 <drawing>
 <settings>
@@
 <part name="J1" library="SparkFun-Connectors" deviceset="POWER_JACK" device=""/>
 <part name="IC1" library="lm1117" deviceset="LM1117MPX-*" device="" technology="5.0"/>
-<part name="U1" library="ST Microelctronics_By_element14_Batch_1" deviceset="STM32L151C6T6" device=""/>
-<part name="JP1" library="pinhead" library_urn="urn:adsk.eagle:library:325" deviceset="PINHD-1X12" device="" package3d_urn="urn:adsk.eagle:package:22487/2"/>
 </parts>
 <sheets>
@@
 <instance part="J1" gate="G$1" x="-33.02" y="165.1"/>
 <instance part="IC1" gate="G$1" x="-30.48" y="147.32"/>
-<instance part="U1" gate="A" x="55.88" y="152.4"/>
-<instance part="JP1" gate="G$1" x="106.68" y="175.26"/>
 </instances>
 <busses>
@@
 </schematic>
 </drawing>
-<compatibility>
-<note version="8.2" severity="warning">
-Since Version 8.2, EAGLE supports online libraries. The ids
-of those online libraries will not be understood (or retained)
-with this version.
-</note>
-<note version="8.3" severity="warning">
-Since Version 8.3, EAGLE supports URNs for individual library
-assets (packages, symbols, and devices). The URNs of those assets
-will not be understood (or retained) with this version.
-</note>
-<note version="8.3" severity="warning">
-Since Version 8.3, EAGLE supports the association of 3D packages
-with devices in libraries, schematics, and board files. Those 3D
-packages will not be understood (or retained) with this version.
-</note>
-</compatibility>
 </eagle>
